File: pcb/lamp-pcb.sch (KiCad schematic (older format))
At the start: 0 parts

Commit message: MCU set up with programming and serial headers
Parts:
- added C? (x2): 20pF, symbol C
- added C? (x5): 0.1uF, symbol C
- added IC?: ATMEGA328P_TQFP, symbol ATMEGA328P_TQFP
- added P?: AVR_ISP, symbol AVR_ISP
- added P?: SERIAL, symbol 6PIN_HEADER
- added Y?: 16MHz, symbol CRYSTAL
Connections:
- new net: C?.2, IC?.20 (AREF)
- new net: C?.2, IC?.7 (XTAL1(PB6)), Y?.1
- new net: C?.2, IC?.8 (XTAL2(PB7)), Y?.2
- new net: C?.2, P?.6
- new net AVR_MISO: IC?.16 (PB4(PCINT4/MISO)), P?.1 (MISO)
- new net AVR_MOSI: IC?.15 (PB3(PCINT3/OC2A/MOSI)), P?.4 (MOSI)
- new net AVR_RST: C?.1, IC?.29 (~RESET~(PC6)), P?.5 (RESET)
- new net AVR_SCK: IC?.17 (PB5(SCK/PCINT5)), P?.3 (SCK)
- new net GND: C?.1, C?.1, C?.1, C?.2, C?.2, C?.2, IC?.21 (GND), IC?.3 (GND), IC?.5 (GND), P?.1, P?.2, P?.6 (GND)
- new net USART_RX: IC?.30 (PD0(RXD/PCINT16)), P?.4
- new net USART_TX: IC?.31 (PD1(TXD/PCINT17)), P?.5
- new net VCC: C?.1, C?.1, C?.1, IC?.18 (AVCC), IC?.4 (VCC), IC?.6 (VCC), P?.2 (VCC), P?.3

Commit message: got an led driver on there
Parts:
- added C?: 0.1uF, symbol C
- added IC?: TLC5971, symbol TLC5971_SOP
- added P?: DCIN, symbol 2PIN_MALE
- added R?: 2.2kΩ, symbol R
- IC?: value ATMEGA328P_TQFP -> ATMEGA328P
Connections:
- net GND: now also C?.1, IC?.0 (PAD), IC?.2 (GND), P?.2, R?.1
- net VCC: now also C?.2, IC?.19 (VCC), IC?.20 (VREG)
- new net: IC?.1 (IREF), R?.2
- new net LED_B0: IC?.5 (OUTB0)
- new net LED_B1: IC?.8 (OUTB1)
- new net LED_B2: IC?.15 (OUTB2)
- new net LED_B3: IC?.18 (OUTB3)
- new net LED_G0: IC?.4 (OUTG0)
- new net LED_G1: IC?.7 (OUTG1)
- new net LED_G2: IC?.14 (OUTG2)
- new net LED_G3: IC?.17 (OUTG3)
- new net LED_MOSI: IC?.9 (SDTI)
- new net LED_R0: IC?.3 (OUTR0)
- new net LED_R1: IC?.6 (OUTR1)
- new net LED_R2: IC?.13 (OUTR2)
- new net LED_R3: IC?.16 (OUTR3)
- new net LED_SCK: IC?.10 (SCKI)
- new net VIN: P?.1
- no-connect marks 0 -> 2
Changed lines of the file:
@@
 P 3550 2600
 F 0 "IC?" H 2850 3750 60  0000 C CNN
-F 1 "ATMEGA328P_TQFP" H 3900 1400 60  0000 C CNN
+F 1 "ATMEGA328P" H 3900 1400 60  0000 C CNN
 F 2 "" H 3550 2600 60  0000 C CNN
 F 3 "" H 3550 2600 60  0000 C CNN
@@
 Wire Wire Line
 	3450 5850 3550 5850
+$Comp
+L TLC5971_SOP IC?
+U 1 1 530E3538
+P 8150 2050
+F 0 "IC?" H 8050 2900 60  0000 C CNN
+F 1 "TLC5971" H 8150 2800 60  0000 C CNN
+F 2 "" H 8150 2050 60  0001 C CNN
+F 3 "" H 8150 2050 60  0001 C CNN
+F 4 "TI" H 7850 1300 60  0001 C CNN "Manufacturer"
+F 5 "TLC5971PWP" H 8250 1300 60  0001 C CNN "Part"
+	1    8150 2050
+	1    0    0    -1
+$EndComp
+$Comp
+L 2PIN_MALE P?
+U 1 1 530E35EB
+P 3700 6700
+F 0 "P?" H 3650 6900 60  0000 C CNN
+F 1 "DCIN" H 3700 6500 60  0000 C CNN
+F 2 "" H 3650 6500 60  0000 C CNN
+F 3 "" H 3650 6500 60  0000 C CNN
+	1    3700 6700
+	1    0    0    -1
+$EndComp
+Text Label 3400 6650 0    60   ~ 0
+VIN
+$Comp
+L GND #PWR?
+U 1 1 530E3694
+P 3450 6750
+F 0 "#PWR?" H 3450 6750 30  0001 C CNN
+F 1 "GND" H 3450 6680 30  0001 C CNN
+F 2 "" H 3450 6750 60  0000 C CNN
+F 3 "" H 3450 6750 60  0000 C CNN
+	1    3450 6750
+	0    1    1    0
+$EndComp
+Wire Wire Line
+	3450 6750 3600 6750
+Wire Wire Line
+	3600 6650 3400 6650
+$Comp
+L C C?
+U 1 1 530E374A
+P 7450 1800
+F 0 "C?" V 7550 2000 60  0000 C CNN
+F 1 "0.1uF" V 7450 2050 60  0000 C CNN
+F 2 "" H 7450 1800 60  0001 C CNN
+F 3 "" H 7450 1800 60  0001 C CNN
+	1    7450 1800
+	0    -1   -1   0
+$EndComp
+$Comp
+L VCC #PWR?
+U 1 1 530E378B
+P 7350 1500
+F 0 "#PWR?" H 7350 1600 30  0001 C CNN
+F 1 "VCC" H 7350 1600 30  0000 C CNN
+F 2 "" H 7350 1500 60  0000 C CNN
+F 3 "" H 7350 1500 60  0000 C CNN
+	1    7350 1500
+	0    -1   -1   0
+$EndComp
+Wire Wire Line
+	7350 1500 7650 1500
+Wire Wire Line
+	7450 1500 7450 1700
+Connection ~ 7450 1500
+Wire Wire Line
+	7450 1700 7650 1700
+Wire Wire Line
+	7200 1900 7650 1900
+$Comp
+L R R?
+U 1 1 530E38F8
+P 7400 2100
+F 0 "R?" H 7100 2000 60  0000 C CNN
+F 1 "2.2kΩ" H 7350 2000 60  0000 C CNN
+F 2 "" H 7400 2100 60  0001 C CNN
+F 3 "" H 7400 2100 60  0001 C CNN
+	1    7400 2100
+	1    0    0    -1
+$EndComp
+$Comp
+L GND #PWR?
+U 1 1 530E395C
+P 7100 2000
+F 0 "#PWR?" H 7100 2000 30  0001 C CNN
+F 1 "GND" H 7100 1930 30  0001 C CNN
+F 2 "" H 7100 2000 60  0000 C CNN
+F 3 "" H 7100 2000 60  0000 C CNN
+	1    7100 2000
+	0    1    1    0
+$EndComp
+Wire Wire Line
+	7100 2000 7200 2000
+Wire Wire Line
+	7200 1900 7200 2100
+Wire Wire Line
+	7200 2100 7250 2100
+Connection ~ 7200 2000
+Connection ~ 7450 1900
+Wire Wire Line
+	7550 2100 7650 2100
+NoConn ~ 7650 2600
+NoConn ~ 7650 2500
+Text Label 7050 2400 0    60   ~ 0
+LED_MOSI
+Text Label 7050 2500 0    60   ~ 0
+LED_SCK
+Wire Wire Line
+	7050 2400 7500 2400
+Wire Wire Line
+	7500 2400 7500 2300
+Wire Wire Line
+	7500 2300 7650 2300
+Wire Wire Line
+	7650 2400 7550 2400
+Wire Wire Line
+	7550 2400 7550 2500
+Wire Wire Line
+	7550 2500 7050 2500
+$Comp
+L GND #PWR?
+U 1 1 530E3B27
+P 8150 2950
+F 0 "#PWR?" H 8150 2950 30  0001 C CNN
+F 1 "GND" H 8150 2880 30  0001 C CNN
+F 2 "" H 8150 2950 60  0000 C CNN
+F 3 "" H 8150 2950 60  0000 C CNN
+	1    8150 2950
+	1    0    0    -1
+$EndComp
+Wire Wire Line
+	8150 2950 8150 2850
+Text Label 9100 1500 2    60   ~ 0
+LED_R0
+Text Label 9100 1600 2    60   ~ 0
+LED_G0
+Text Label 9100 1700 2    60   ~ 0
+LED_B0
+Text Label 9100 1800 2    60   ~ 0
+LED_R1
+Text Label 9100 1900 2    60   ~ 0
+LED_G1
+Text Label 9100 2000 2    60   ~ 0
+LED_B1
+Text Label 9100 2100 2    60   ~ 0
+LED_R2
+Text Label 9100 2200 2    60   ~ 0
+LED_G2
+Text Label 9100 2300 2    60   ~ 0
+LED_B2
+Text Label 9100 2400 2    60   ~ 0
+LED_R3
+Text Label 9100 2500 2    60   ~ 0
+LED_G3
+Text Label 9100 2600 2    60   ~ 0
+LED_B3
+Wire Wire Line
+	9100 1500 8650 1500
+Wire Wire Line
+	8650 1600 9100 1600
+Wire Wire Line
+	9100 1700 8650 1700
+Wire Wire Line
+	8650 1800 9100 1800
+Wire Wire Line
+	9100 1900 8650 1900
+Wire Wire Line
+	8650 2000 9100 2000
+Wire Wire Line
+	9100 2100 8650 2100
+Wire Wire Line
+	8650 2200 9100 2200
+Wire Wire Line
+	9100 2300 8650 2300
+Wire Wire Line
+	8650 2400 9100 2400
+Wire Wire Line
+	9100 2500 8650 2500
+Wire Wire Line
+	8650 2600 9100 2600
 $EndSCHEMATC

Commit message: put a basic volatge regulator on there. may switch it out for something else
Parts:
- added C?: 10uF, symbol C_POL
- added C?: 22uF, symbol C_POL
- added IC?: LM1117, symbol LM1117
Connections:
- net GND: now also C?.2, C?.2, IC?.1 (ADJ/GND)
- net VCC: now also C?.1, IC?.0 (VOUT), IC?.2 (VOUT)
- net VIN: now also C?.1, IC?.3 (VIN)
Other:
- moved on the sheet: P?
Changed lines of the file:
@@
 L 2PIN_MALE P?
 U 1 1 530E35EB
-P 3700 6700
-F 0 "P?" H 3650 6900 60  0000 C CNN
-F 1 "DCIN" H 3700 6500 60  0000 C CNN
-F 2 "" H 3650 6500 60  0000 C CNN
-F 3 "" H 3650 6500 60  0000 C CNN
-	1    3700 6700
-	1    0    0    -1
-$EndComp
-Text Label 3400 6650 0    60   ~ 0
+P 6550 4350
+F 0 "P?" H 6500 4550 60  0000 C CNN
+F 1 "DCIN" H 6550 4150 60  0000 C CNN
+F 2 "" H 6500 4150 60  0000 C CNN
+F 3 "" H 6500 4150 60  0000 C CNN
+	1    6550 4350
+	1    0    0    -1
+$EndComp
+Text Label 6250 4300 0    60   ~ 0
 VIN
 $Comp
 L GND #PWR?
 U 1 1 530E3694
-P 3450 6750
-F 0 "#PWR?" H 3450 6750 30  0001 C CNN
-F 1 "GND" H 3450 6680 30  0001 C CNN
-F 2 "" H 3450 6750 60  0000 C CNN
-F 3 "" H 3450 6750 60  0000 C CNN
-	1    3450 6750
-	0    1    1    0
-$EndComp
-Wire Wire Line
-	3450 6750 3600 6750
-Wire Wire Line
-	3600 6650 3400 6650
+P 6300 4400
+F 0 "#PWR?" H 6300 4400 30  0001 C CNN
+F 1 "GND" H 6300 4330 30  0001 C CNN
+F 2 "" H 6300 4400 60  0000 C CNN
+F 3 "" H 6300 4400 60  0000 C CNN
+	1    6300 4400
+	0    1    1    0
+$EndComp
+Wire Wire Line
+	6300 4400 6450 4400
+Wire Wire Line
+	6450 4300 6250 4300
 $Comp
 L C C?
@@
 Wire Wire Line
 	8650 2600 9100 2600
+$Comp
+L LM1117 IC?
+U 1 1 530E4152
+P 8100 4350
+F 0 "IC?" H 7900 4750 60  0000 C CNN
+F 1 "LM1117" H 8000 4650 60  0000 C CNN
+F 2 "" H 8100 4350 60  0000 C CNN
+F 3 "" H 8100 4350 60  0000 C CNN
+	1    8100 4350
+	1    0    0    -1
+$EndComp
+$Comp
+L GND #PWR?
+U 1 1 530E4235
+P 7550 4250
+F 0 "#PWR?" H 7550 4250 30  0001 C CNN
+F 1 "GND" H 7550 4180 30  0001 C CNN
+F 2 "" H 7550 4250 60  0000 C CNN
+F 3 "" H 7550 4250 60  0000 C CNN
+	1    7550 4250
+	0    1    1    0
+$EndComp
+$Comp
+L VCC #PWR?
+U 1 1 530E4249
+P 7350 4250
+F 0 "#PWR?" H 7350 4350 30  0001 C CNN
+F 1 "VCC" H 7350 4350 30  0000 C CNN
+F 2 "" H 7350 4250 60  0000 C CNN
+F 3 "" H 7350 4250 60  0000 C CNN
+	1    7350 4250
+	1    0    0    -1
+$EndComp
+Text Label 7350 4450 0    60   ~ 0
+VIN
+Wire Wire Line
+	7350 4450 7650 4450
+Wire Wire Line
+	7650 4350 7350 4350
+Wire Wire Line
+	7350 4350 7350 4250
+Wire Wire Line
+	7650 4250 7550 4250
+$Comp
+L VCC #PWR?
+U 1 1 530E4380
+P 8650 4350
+F 0 "#PWR?" H 8650 4450 30  0001 C CNN
+F 1 "VCC" H 8650 4450 30  0000 C CNN
+F 2 "" H 8650 4350 60  0000 C CNN
+F 3 "" H 8650 4350 60  0000 C CNN
+	1    8650 4350
+	0    1    1    0
+$EndComp
+Wire Wire Line
+	8650 4350 8550 4350
+$Comp
+L C_POL C?
+U 1 1 530E44C1
+P 7550 4650
+F 0 "C?" V 7550 4450 60  0000 C CNN
+F 1 "10uF" V 7650 4450 60  0000 C CNN
+F 2 "" H 7550 4650 60  0001 C CNN
+F 3 "" H 7550 4650 60  0001 C CNN
+	1    7550 4650
+	0    1    1    0
+$EndComp
+$Comp
+L C_POL C?
+U 1 1 530E44E9
+P 8600 4550
+F 0 "C?" V 8600 4700 60  0000 C CNN
+F 1 "22uF" V 8700 4750 60  0000 C CNN
+F 2 "" H 8600 4550 60  0001 C CNN
+F 3 "" H 8600 4550 60  0001 C CNN
+	1    8600 4550
+	0    1    1    0
+$EndComp
+$Comp
+L GND #PWR?
+U 1 1 530E4552
+P 7550 4850
+F 0 "#PWR?" H 7550 4850 30  0001 C CNN
+F 1 "GND" H 7550 4780 30  0001 C CNN
+F 2 "" H 7550 4850 60  0000 C CNN
+F 3 "" H 7550 4850 60  0000 C CNN
+	1    7550 4850
+	1    0    0    -1
+$EndComp
+$Comp
+L GND #PWR?
+U 1 1 530E4566
+P 8600 4750
+F 0 "#PWR?" H 8600 4750 30  0001 C CNN
+F 1 "GND" H 8600 4680 30  0001 C CNN
+F 2 "" H 8600 4750 60  0000 C CNN
+F 3 "" H 8600 4750 60  0000 C CNN
+	1    8600 4750
+	1    0    0    -1
+$EndComp
+Wire Wire Line
+	8600 4750 8600 4650
+Wire Wire Line
+	7550 4850 7550 4750
+Wire Wire Line
+	7550 4550 7550 4450
+Connection ~ 7550 4450
+Wire Wire Line
+	8600 4450 8600 4350
+Connection ~ 8600 4350
 $EndSCHEMATC

Commit message: first pass at schematic done
Parts:
- removed C?: 0.1uF, symbol C
- removed IC?: TLC5971, symbol TLC5971_SOP
- removed R?: 2.2kΩ, symbol R
- added C10, C11: 0.1uF, symbol C
- added IC3: TLC5973, symbol TLC5973
- added J1: 7-12V_OUT, symbol 2PIN_FEMALE
- added J2: LED_CARD_BOTTOM, symbol 5PIN_FEMALE
- added LED1, LED2: RGB-CA, symbol LED_RGB-CA
- added P4, P5, P6: LEDSTACK, symbol 5PIN_MALE
- added P7: LED_CARD_TOP, symbol 5PIN_MALE
- added R1, R2, R3: 10kΩ, symbol R
- added R4: 2kΩ, symbol R
- added R5: 1kΩ, symbol R
- added S1: TOP, symbol SPDT
- P1: renamed from P?; value DCIN -> 7-12V_IN
- gave numbers to parts that had none: 14
Connections:
- net GND: now also J1.2, P4.3, P5.3, P6.3, R1.2, R2.2, R3.2, R4.2
- net VCC: now also P4.2, P5.2, P6.2
- net VIN: now also J1.1, P4.1, P5.1, P6.1
- net LEDSTACK1: now reaches IC1.1 (PD3(PCINT19/OC2B/INT1))
- net LEDSTACK1: now also P5.4
- net LEDSTACK2: now reaches IC1.2 (PD4(PCINT20/XCK/T0))
- net LEDSTACK2: now also P6.4
- net STACKSENSE0: now reaches IC1.23 (PC0(ADC0/PCINT8))
- net STACKSENSE0: now also P4.5, R3.1
- net STACKSENSE1: now reaches IC1.24 (PC1(ADC1/PCINT9))
- net STACKSENSE1: now also P5.5, R2.1
- net STACKSENSE2: now reaches IC1.25 (PC2(ADC2/PCINT10))
- net STACKSENSE2: now also P6.5, R1.1
- net LEDSTACK0: now reaches IC1.32 (PD2(INT0/PCINT18))
- net LEDSTACK0: now also P4.4
- new net: IC3.7 (IREF), R4.1
- new net BLU: IC3.3 (OUT2), LED1.4 (B), LED2.4 (B)
- new net GRN: IC3.2 (OUT1), LED1.3 (G), LED2.3 (G)
- new net LED_GND: C10.1, C11.2, IC3.4 (GND), J2.3, P7.3
- new net LED_SER_IN: IC3.6 (SDI), J2.4
- new net LED_SER_OUT: IC3.5 (SDO), P7.4
- new net RED: IC3.1 (OUT0), LED1.1 (R), LED2.1 (R)
- new net SENSE_BOT: J2.5, R5.1
- new net SENSE_TOP: P7.5, R5.2, S1.3
- new net VLED: C11.1, J2.1, LED1.2 (A), LED2.2 (A), P7.1
- new net VLOG: C10.2, IC3.8 (VCC), J2.2, S1.2 (COM)
- new net VLOG_TOP: P7.2, S1.1
- no-connect marks 2 -> 11
Other:
- note added: "7-12 V Input/Output and 5V Regulator"
- note added: "LED Board (Multiple)"
- note added: "LED Stack Headers"
- note added: "MCU"
- note added: "Programming and Communication Headers"
- moved on the sheet: C1, C2, C3, C4, C5, C6, C7, C8, C9, IC1, IC2, P1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
