File: pcb/lamp-expansion/lamp-expansion.kicad_pcb (KiCad board)
At the start: 2 copper layers, 139.7 x 46.2 mm, 77 parts, among them IC1 PAM2421, IC2 MCP73811, IC3 NTHD3101F, IC6 LM1117_5.0, IC7 FT230X_SOP, IC9 CC3000, J1 MICROUSB, J2 DCIN, J3 SERIAL, J4 5PIN_INPUT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

Commit message: last few traces
Routing:
- net VCC: track 4.93 -> 76.3 mm, vias 0 -> 2
- net GND: track 100.3 -> 161.8 mm, vias 17 -> 61
- net /POT_0: track 2.54 -> 38.3 mm, vias 0 -> 3
- net /CC_MOSI: track 34.6 -> 26.4 mm
- net /CC_SEL: track 31.0 -> 35.6 mm
- net /CC_EN: track 43.8 -> 46.5 mm
- net /CC_SCK: track 20.5 -> 22.7 mm
- net /CC_MISO: track 37.8 -> 36.4 mm
- net /CC_IRQ: track 30.6 -> 31.2 mm

Commit message: safety commit
Parts:
- moved R10 0.64 mm to (179.1, 113.0), turned to 180 degrees
Routing:
- net GND: track 161.8 -> 214.9 mm, vias 61 -> 78
- net VCC: track 76.3 -> 86.9 mm, vias 2 -> 0
- net /CC_EN: track 46.5 -> 45.5 mm, vias 0 -> 2
Other:
- net class POWER added: clearance 0.2032, trace_width 0.889, via_dia 0.762, via_drill 0.381
- net class RF added: clearance 0.2032, trace_width 0.889, via_dia 0.762, via_drill 0.381
